File: kicad/safeduino_mega_2560.sch (KiCad schematic (older format))
At the start: 106 parts, among them X1 USB

Commit message: Продолжил переделывать проект.
Parts:
- XP16, XP20, XP21, XP26, XP27, XP28, XP29, XP32, XP36, XP37, XP38, XP39, XP40, XP41, XP42, XP48, XP53, XP54, XP55, XP56, XP57, XP58, XP59, XP60, XP61, XP62, XP65, XP67, XP68, XP7: footprint ~ -> IWconnectors:1_pin
Changed lines of the file:
@@
 F 0 "XP7" H 17775 13725 50  0000 L BNN
 F 1 "~" H 17400 13850 50  0000 L BNN
-F 2 "~" H 17800 13900 50  0001 C CNN
+F 2 "IWconnectors:1_pin" H 17800 13900 50  0001 C CNN
 F 3 "" H 17350 13750 60  0001 C CNN
 	1    17350 13750
@@
 F 0 "XP16" H 16475 12525 50  0000 L BNN
 F 1 "~" H 16100 12650 50  0000 L BNN
-F 2 "~" H 16500 12700 50  0001 C CNN
+F 2 "IWconnectors:1_pin" H 16500 12700 50  0001 C CNN
 F 3 "" H 16050 12550 60  0001 C CNN
 	1    16050 12550
@@
 F 0 "XP21" H 15225 12625 50  0000 L BNN
 F 1 "~" H 14850 12750 50  0000 L BNN
-F 2 "~" H 15250 12800 50  0001 C CNN
+F 2 "IWconnectors:1_pin" H 15250 12800 50  0001 C CNN
 F 3 "" H 14800 12650 60  0001 C CNN
 	1    14800 12650
@@
 F 0 "XP20" H 15225 12525 50  0000 L BNN
 F 1 "~" H 14850 12650 50  0000 L BNN
-F 2 "~" H 15250 12700 50  0001 C CNN
+F 2 "IWconnectors:1_pin" H 15250 12700 50  0001 C CNN
 F 3 "" H 14800 12550 60  0001 C CNN
 	1    14800 12550
@@
 F 0 "XP28" H 15225 13175 50  0000 L BNN
 F 1 "~" H 14850 13300 50  0000 L BNN
-F 2 "~" H 15250 13350 50  0001 C CNN
+F 2 "IWconnectors:1_pin" H 15250 13350 50  0001 C CNN
 F 3 "" H 14800 13200 60  0001 C CNN
 	1    14800 13200
@@
 F 0 "XP29" H 15225 13275 50  0000 L BNN
 F 1 "~" H 14850 13400 50  0000 L BNN
-F 2 "~" H 15250 13450 50  0001 C CNN
+F 2 "IWconnectors:1_pin" H 15250 13450 50  0001 C CNN
 F 3 "" H 14800 13300 60  0001 C CNN
 	1    14800 13300
@@
 F 0 "XP27" H 15225 13075 50  0000 L BNN
 F 1 "~" H 14850 13200 50  0000 L BNN
-F 2 "~" H 15250 13250 50  0001 C CNN
+F 2 "IWconnectors:1_pin" H 15250 13250 50  0001 C CNN
 F 3 "" H 14800 13100 60  0001 C CNN
 	1    14800 13100
@@
 F 0 "XP26" H 15225 12975 50  0000 L BNN
 F 1 "~" H 14850 13100 50  0000 L BNN
-F 2 "~" H 15250 13150 50  0001 C CNN
+F 2 "IWconnectors:1_pin" H 15250 13150 50  0001 C CNN
 F 3 "" H 14800 13000 60  0001 C CNN
 	1    14800 13000
@@
 F 0 "XP42" H 16475 13525 50  0000 L BNN
 F 1 "~" H 16100 13650 50  0000 L BNN
-F 2 "~" H 16500 13700 50  0001 C CNN
+F 2 "IWconnectors:1_pin" H 16500 13700 50  0001 C CNN
 F 3 "" H 16050 13550 60  0001 C CNN
 	1    16050 13550
@@
 F 0 "XP41" H 16475 13425 50  0000 L BNN
 F 1 "~" H 16100 13550 50  0000 L BNN
-F 2 "~" H 16500 13600 50  0001 C CNN
+F 2 "IWconnectors:1_pin" H 16500 13600 50  0001 C CNN
 F 3 "" H 16050 13450 60  0001 C CNN
 	1    16050 13450
@@
 F 0 "XP38" H 16475 13325 50  0000 L BNN
 F 1 "~" H 16100 13450 50  0000 L BNN
-F 2 "~" H 16500 13500 50  0001 C CNN
+F 2 "IWconnectors:1_pin" H 16500 13500 50  0001 C CNN
 F 3 "" H 16050 13350 60  0001 C CNN
 	1    16050 13350
@@
 F 0 "XP48" H 16475 13825 50  0000 L BNN
 F 1 "~" H 16100 13950 50  0000 L BNN
-F 2 "~" H 16500 14000 50  0001 C CNN
+F 2 "IWconnectors:1_pin" H 16500 14000 50  0001 C CNN
 F 3 "" H 16050 13850 60  0001 C CNN
 	1    16050 13850
@@
 F 0 "XP53" H 16475 13925 50  0000 L BNN
 F 1 "~" H 16100 14050 50  0000 L BNN
-F 2 "~" H 16500 14100 50  0001 C CNN
+F 2 "IWconnectors:1_pin" H 16500 14100 50  0001 C CNN
 F 3 "" H 16050 13950 60  0001 C CNN
 	1    16050 13950
@@
 F 0 "XP54" H 17775 12525 50  0000 L BNN
 F 1 "~" H 17400 12650 50  0000 L BNN
-F 2 "~" H 17800 12700 50  0001 C CNN
+F 2 "IWconnectors:1_pin" H 17800 12700 50  0001 C CNN
 F 3 "" H 17350 12550 60  0001 C CNN
 	1    17350 12550
@@
 F 0 "XP55" H 17775 12625 50  0000 L BNN
 F 1 "~" H 17400 12750 50  0000 L BNN
-F 2 "~" H 17800 12800 50  0001 C CNN
+F 2 "IWconnectors:1_pin" H 17800 12800 50  0001 C CNN
 F 3 "" H 17350 12650 60  0001 C CNN
 	1    17350 12650
@@
 F 0 "XP57" H 17775 12825 50  0000 L BNN
 F 1 "~" H 17400 12950 50  0000 L BNN
-F 2 "~" H 17800 13000 50  0001 C CNN
+F 2 "IWconnectors:1_pin" H 17800 13000 50  0001 C CNN
 F 3 "" H 17350 12850 60  0001 C CNN
 	1    17350 12850
@@
 F 0 "XP56" H 17775 12725 50  0000 L BNN
 F 1 "~" H 17400 12850 50  0000 L BNN
-F 2 "~" H 17800 12900 50  0001 C CNN
+F 2 "IWconnectors:1_pin" H 17800 12900 50  0001 C CNN
 F 3 "" H 17350 12750 60  0001 C CNN
 	1    17350 12750
@@
 F 0 "XP60" H 17775 13125 50  0000 L BNN
 F 1 "~" H 17400 13250 50  0000 L BNN
-F 2 "~" H 17800 13300 50  0001 C CNN
+F 2 "IWconnectors:1_pin" H 17800 13300 50  0001 C CNN
 F 3 "" H 17350 13150 60  0001 C CNN
 	1    17350 13150
@@
 F 0 "XP61" H 17775 13225 50  0000 L BNN
 F 1 "~" H 17400 13350 50  0000 L BNN
-F 2 "~" H 17800 13400 50  0001 C CNN
+F 2 "IWconnectors:1_pin" H 17800 13400 50  0001 C CNN
 F 3 "" H 17350 13250 60  0001 C CNN
 	1    17350 13250
@@
 F 0 "XP59" H 17775 13025 50  0000 L BNN
 F 1 "~" H 17400 13150 50  0000 L BNN
-F 2 "~" H 17800 13200 50  0001 C CNN
+F 2 "IWconnectors:1_pin" H 17800 13200 50  0001 C CNN
 F 3 "" H 17350 13050 60  0001 C CNN
 	1    17350 13050
@@
 F 0 "XP58" H 17775 12925 50  0000 L BNN
 F 1 "~" H 17400 13050 50  0000 L BNN
-F 2 "~" H 17800 13100 50  0001 C CNN
+F 2 "IWconnectors:1_pin" H 17800 13100 50  0001 C CNN
 F 3 "" H 17350 12950 60  0001 C CNN
 	1    17350 12950
@@
 F 0 "XP37" H 16475 13025 50  0000 L BNN
 F 1 "~" H 16100 13150 50  0000 L BNN
-F 2 "~" H 16500 13200 50  0001 C CNN
+F 2 "IWconnectors:1_pin" H 16500 13200 50  0001 C CNN
 F 3 "" H 16050 13050 60  0001 C CNN
 	1    16050 13050
@@
 F 0 "XP36" H 16475 12925 50  0000 L BNN
 F 1 "~" H 16100 13050 50  0000 L BNN
-F 2 "~" H 16500 13100 50  0001 C CNN
+F 2 "IWconnectors:1_pin" H 16500 13100 50  0001 C CNN
 F 3 "" H 16050 12950 60  0001 C CNN
 	1    16050 12950
@@
 F 0 "XP32" H 16475 12825 50  0000 L BNN
 F 1 "~" H 16100 12950 50  0000 L BNN
-F 2 "~" H 16500 13000 50  0001 C CNN
+F 2 "IWconnectors:1_pin" H 16500 13000 50  0001 C CNN
 F 3 "" H 16050 12850 60  0001 C CNN
 	1    16050 12850
@@
 F 0 "XP67" H 19750 14200 50  0000 L BNN
 F 1 "~" H 19650 14200 50  0000 L BNN
-F 2 "~" H 20050 14250 50  0001 C CNN
+F 2 "IWconnectors:1_pin" H 20050 14250 50  0001 C CNN
 F 3 "" H 19600 14100 60  0001 C CNN
 	1    19600 14100
@@
 F 0 "XP68" H 19750 14450 50  0000 L BNN
 F 1 "~" H 19650 14450 50  0000 L BNN
-F 2 "~" H 20050 14500 50  0001 C CNN
+F 2 "IWconnectors:1_pin" H 20050 14500 50  0001 C CNN
 F 3 "" H 19600 14350 60  0001 C CNN
 	1    19600 14350
@@
 F 0 "XP40" H 19750 11700 50  0000 L BNN
 F 1 "~" H 19650 11700 50  0000 L BNN
-F 2 "~" H 20050 11750 50  0001 C CNN
+F 2 "IWconnectors:1_pin" H 20050 11750 50  0001 C CNN
 F 3 "" H 19600 11600 60  0001 C CNN
 	1    19600 11600
@@
 F 0 "XP39" H 19750 11450 50  0000 L BNN
 F 1 "~" H 19650 11450 50  0000 L BNN
-F 2 "~" H 20050 11500 50  0001 C CNN
+F 2 "IWconnectors:1_pin" H 20050 11500 50  0001 C CNN
 F 3 "" H 19600 11350 60  0001 C CNN
 	1    19600 11350
@@
 F 0 "XP65" H 17775 13625 50  0000 L BNN
 F 1 "~" H 17400 13750 50  0000 L BNN
-F 2 "~" H 17800 13800 50  0001 C CNN
+F 2 "IWconnectors:1_pin" H 17800 13800 50  0001 C CNN
 F 3 "" H 17350 13650 60  0001 C CNN
 	1    17350 13650
@@
 F 0 "XP62" H 17775 13525 50  0000 L BNN
 F 1 "~" H 17400 13650 50  0000 L BNN
-F 2 "~" H 17800 13700 50  0001 C CNN
+F 2 "IWconnectors:1_pin" H 17800 13700 50  0001 C CNN
 F 3 "" H 17350 13550 60  0001 C CNN
 	1    17350 13550

Commit message: Приступил к переработке платы SafeDuino MEGA 2560.
Parts:
- removed X1: USB, IWconnectors:CONN_USB-B, symbol LFconnectors:USB
- removed XP20, XP21, XP29, XP38, XP41, XP42, XP54, XP55, XP56, XP57, XP58, XP59, XP60, XP61: ~, IWconnectors:1_pin, symbol LFconnectors:PIN_M_1
- added VD10, VD7, VD9: PESD5V0L1BA,115, IWcomponents:SOD323, symbol LFdiod:STABILITRON_TWO
- added VD8: SS14, IWcomponents:SMA, symbol LFdiod:SHOTTKY_DIODE
- added X1: USBB-1J, IWconnectors:CONN_USB-B, symbol LFconnectors:connector_6pin_gost
- added XS10: 2214SM-36G-75-PCP, IWconnectors:PIN_ARRAY_18x2, symbol LFconnectors:connector_36pin_gost
- S1: value DTSGL-61K -> FSM1LP
Connections:
- net labels added: PB0, PB1, PB2, PB3, UD+, UD-
- wire segments 484 -> 524
Other:
- note added: "+5 V"
- note added: "D+"
- note added: "D-"
- note added: "MISO"
- note added: "MOSI"
- note added: "PA0"
- note added: "PA1"
- note added: "PA2"
- note added: "PA3"
- note added: "PA4"
- note added: "PA5"
- note added: "PA6"
- note added: "PA7"
- note added: "PC0"
- note added: "PC1"
- note added: "PC2"
- note added: "PC3"
- note added: "PC4"
- note added: "PC5"
- note added: "PC6"
- note added: "PC7"
- note added: "PD7"
- note added: "PG0"
- note added: "PG1"
- note added: "PG2"
- note added: "PL0"
- note added: "PL1"
- note added: "PL2"
- note added: "PL3"
- note added: "PL4"
- note added: "PL5"
- note added: "PL6"
- note added: "PL7"
- note added: "SCK"
- note added: "SS"
- note added: "Shield"
- note added: "Vbus"
- note added: "Vin"
- note added: "Vmpu"
- note added: "Vusb"
- note added: "Внешнее\nпитание +5В"
- note added: "Перемычка для переключения\n между внешним питанием и\n питанием от USB"
- note removed: "PC"
- note removed: "PG"
- note removed: "PL"
- moved on the sheet: C1, C10, C11, C12, C13, C14, C15, C16, C17, C18, C19, C2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
