File: kicad/safeduino_mega_2560.sch (KiCad schematic (older format))
At the start: 80 parts, among them X1 USBB-1J

Commit message: Закончил предварительную трассировку платы.
Changed lines of the file:
@@
 	19600 9050 20000 9050
 Wire Wire Line
-	18450 7400 18550 7400
-Connection ~ 18450 7400
-Wire Wire Line
-	18450 7300 18450 7400
-Wire Wire Line
-	18550 7300 18450 7300
-Wire Wire Line
-	18000 7400 18450 7400
-Text Notes 18950 6050 0    60   ~ 0
+	19900 3800 20000 3800
+Connection ~ 19900 3800
+Wire Wire Line
+	19900 3700 19900 3800
+Wire Wire Line
+	20000 3700 19900 3700
+Wire Wire Line
+	19450 3800 19900 3800
+Text Notes 20400 2450 0    60   ~ 0
 PG0
-Text Notes 18950 5850 0    60   ~ 0
+Text Notes 20400 2250 0    60   ~ 0
 PG2
-Text Notes 18950 7450 0    60   ~ 0
+Text Notes 20400 3850 0    60   ~ 0
 GND
-Text Notes 18950 7350 0    60   ~ 0
+Text Notes 20400 3750 0    60   ~ 0
 GND
-Text Notes 18950 6850 0    60   ~ 0
+Text Notes 20400 3250 0    60   ~ 0
 PL0
-Text Notes 18950 6750 0    60   ~ 0
+Text Notes 20400 3150 0    60   ~ 0
 PL1
-Text Notes 18950 6650 0    60   ~ 0
+Text Notes 20400 3050 0    60   ~ 0
 PL2
-Text Notes 18950 6550 0    60   ~ 0
+Text Notes 20400 2950 0    60   ~ 0
 PL3
-Text Notes 18950 6450 0    60   ~ 0
+Text Notes 20400 2850 0    60   ~ 0
 PL4
-Text Notes 18950 6350 0    60   ~ 0
+Text Notes 20400 2750 0    60   ~ 0
 PL5
-Text Notes 18950 6250 0    60   ~ 0
+Text Notes 20400 2650 0    60   ~ 0
 PL6
-Text Notes 18950 6150 0    60   ~ 0
+Text Notes 20400 2550 0    60   ~ 0
 PL7
-Text Notes 18950 5950 0    60   ~ 0
+Text Notes 20400 2350 0    60   ~ 0
 PG1
-Text Notes 18950 5750 0    60   ~ 0
+Text Notes 20400 2150 0    60   ~ 0
 PD7
-Text Notes 18950 5650 0    60   ~ 0
+Text Notes 20400 2050 0    60   ~ 0
 PC0
-Text Notes 18950 5550 0    60   ~ 0
+Text Notes 20400 1950 0    60   ~ 0
 PC1
-Text Notes 18950 6950 0    60   ~ 0
+Text Notes 20400 3350 0    60   ~ 0
 MISO
-Text Notes 18950 7050 0    60   ~ 0
+Text Notes 20400 3450 0    60   ~ 0
 MOSI
-Text Notes 18950 7250 0    60   ~ 0
+Text Notes 20400 3650 0    60   ~ 0
 SS
-Text Notes 18950 7150 0    60   ~ 0
+Text Notes 20400 3550 0    60   ~ 0
 SCK
-Text Notes 18950 5450 0    60   ~ 0
+Text Notes 20400 1850 0    60   ~ 0
 PC2
-Text Notes 18950 5350 0    60   ~ 0
+Text Notes 20400 1750 0    60   ~ 0
 PC3
-Text Notes 18950 4950 0    60   ~ 0
+Text Notes 20400 1350 0    60   ~ 0
 PC7
-Text Notes 18950 5050 0    60   ~ 0
+Text Notes 20400 1450 0    60   ~ 0
 PC6
-Text Notes 18950 5250 0    60   ~ 0
+Text Notes 20400 1650 0    60   ~ 0
 PC4
-Text Notes 18950 5150 0    60   ~ 0
+Text Notes 20400 1550 0    60   ~ 0
 PC5
-Connection ~ 18450 4700
-Text Label 18000 4700 0    60   ~ 0
+Connection ~ 19900 1100
+Text Label 19450 1100 0    60   ~ 0
 MPU_VCC
 Wire Wire Line
-	18450 4800 18450 4700
-Wire Wire Line
-	18550 4800 18450 4800
-Text Label 18000 7400 0    60   ~ 0
+	19900 1200 19900 1100
+Wire Wire Line
+	20000 1200 19900 1200
+Text Label 19450 3800 0    60   ~ 0
 GND
 Wire Wire Line
-	18550 7200 18000 7200
-Wire Wire Line
-	18550 7100 18000 7100
-Wire Wire Line
-	18550 7000 18000 7000
-Wire Wire Line
-	18550 6900 18000 6900
-Wire Wire Line
-	18550 6800 18000 6800
-Text Label 18000 6800 0    60   ~ 0
+	20000 3600 19450 3600
+Wire Wire Line
+	20000 3500 19450 3500
+Wire Wire Line
+	20000 3400 19450 3400
+Wire Wire Line
+	20000 3300 19450 3300
+Wire Wire Line
+	20000 3200 19450 3200
+Text Label 19450 3200 0    60   ~ 0
 PL0
 Wire Wire Line
-	18550 6700 18000 6700
-Text Label 18000 6700 0    60   ~ 0
+	20000 3100 19450 3100
+Text Label 19450 3100 0    60   ~ 0
 PL1
 Wire Wire Line
-	18550 6600 18000 6600
-Text Label 18000 6600 0    60   ~ 0
+	20000 3000 19450 3000
+Text Label 19450 3000 0    60   ~ 0
 PL2
 Wire Wire Line
-	18550 6500 18000 6500
-Text Label 18000 6500 0    60   ~ 0
+	20000 2900 19450 2900
+Text Label 19450 2900 0    60   ~ 0
 PL3
 Wire Wire Line
-	18550 6400 18000 6400
-Text Label 18000 6400 0    60   ~ 0
+	20000 2800 19450 2800
+Text Label 19450 2800 0    60   ~ 0
 PL4
 Wire Wire Line
-	18550 6300 18000 6300
-Text Label 18000 6300 0    60   ~ 0
+	20000 2700 19450 2700
+Text Label 19450 2700 0    60   ~ 0
 PL5
-Text Label 18000 6200 0    60   ~ 0
+Text Label 19450 2600 0    60   ~ 0
 PL6
-Text Label 18000 6100 0    60   ~ 0
+Text Label 19450 2500 0    60   ~ 0
 PL7
-Text Label 18000 6000 0    60   ~ 0
+Text Label 19450 2400 0    60   ~ 0
 PG0
-Text Label 18000 5900 0    60   ~ 0
+Text Label 19450 2300 0    60   ~ 0
 PG1
-Text Label 18000 5800 0    60   ~ 0
+Text Label 19450 2200 0    60   ~ 0
 PG2
-Text Label 18000 5700 0    60   ~ 0
+Text Label 19450 2100 0    60   ~ 0
 PD7
-Text Label 18000 5600 0    60   ~ 0
+Text Label 19450 2000 0    60   ~ 0
 PC0
-Text Label 18000 5500 0    60   ~ 0
+Text Label 19450 1900 0    60   ~ 0
 PC1
-Text Label 18000 5400 0    60   ~ 0
+Text Label 19450 1800 0    60   ~ 0
 PC2
-Text Label 18000 5300 0    60   ~ 0
+Text Label 19450 1700 0    60   ~ 0
 PC3
-Text Label 18000 5200 0    60   ~ 0
+Text Label 19450 1600 0    60   ~ 0
 PC4
-Text Label 18000 5100 0    60   ~ 0
+Text Label 19450 1500 0    60   ~ 0
 PC5
-Text Label 18000 5000 0    60   ~ 0
+Text Label 19450 1400 0    60   ~ 0
 PC6
-Text Label 18000 4900 0    60   ~ 0
+Text Label 19450 1300 0    60   ~ 0
 PC7
 Wire Wire Line
-	18550 4700 18450 4700
+	20000 1100 19900 1100
 $Comp
 L LFtransformator:INDUCTOR LL1
@@
 PE2
 Wire Wire Line
-	18000 6200 18550 6200
-Wire Wire Line
-	18000 5300 18550 5300
-Wire Wire Line
-	18000 5200 18550 5200
-Wire Wire Line
-	18000 5100 18550 5100
-Wire Wire Line
-	18000 5000 18550 5000
-Wire Wire Line
-	18000 4900 18550 4900
-Wire Wire Line
-	18000 6100 18550 6100
-Wire Wire Line
-	18000 4700 18450 4700
-Wire Wire Line
-	18000 6000 18550 6000
-Wire Wire Line
-	18000 5900 18550 5900
-Wire Wire Line
-	18000 5800 18550 5800
-Wire Wire Line
-	18000 5700 18550 5700
-Wire Wire Line
-	18000 5600 18550 5600
-Wire Wire Line
-	18000 5500 18550 5500
-Wire Wire Line
-	18000 5400 18550 5400
+	19450 2600 20000 2600
+Wire Wire Line
+	19450 1700 20000 1700
+Wire Wire Line
+	19450 1600 20000 1600
+Wire Wire Line
+	19450 1500 20000 1500
+Wire Wire Line
+	19450 1400 20000 1400
+Wire Wire Line
+	19450 1300 20000 1300
+Wire Wire Line
+	19450 2500 20000 2500
+Wire Wire Line
+	19450 1100 19900 1100
+Wire Wire Line
+	19450 2400 20000 2400
+Wire Wire Line
+	19450 2300 20000 2300
+Wire Wire Line
+	19450 2200 20000 2200
+Wire Wire Line
+	19450 2100 20000 2100
+Wire Wire Line
+	19450 2000 20000 2000
+Wire Wire Line
+	19450 1900 20000 1900
+Wire Wire Line
+	19450 1800 20000 1800
 Text Notes 20400 8500 0    60   ~ 0
 PH7
@@
 Text Notes 20400 9100 0    60   ~ 0
 PE6
-Text Label 18000 7000 0    60   ~ 0
+Text Label 19450 3400 0    60   ~ 0
 MOSI
-Text Label 18000 6900 0    60   ~ 0
+Text Label 19450 3300 0    60   ~ 0
 MISO
-Text Label 18000 7100 0    60   ~ 0
+Text Label 19450 3500 0    60   ~ 0
 SCK
-Text Label 18000 7200 0    60   ~ 0
+Text Label 19450 3600 0    60   ~ 0
 SS
-Text Notes 18950 4850 0    60   ~ 0
+Text Notes 20400 1250 0    60   ~ 0
 +5V
-Text Notes 18950 4750 0    60   ~ 0
+Text Notes 20400 1150 0    60   ~ 0
 +5V
 $Comp
 L LFconnectors:connector_28pin_gost XS10
 U 1 1 64EB12AA
-P 18550 4700
-F 0 "XS10" H 18800 5050 71  0000 L CNN
-F 1 "PBD-28" H 18700 4950 71  0000 L CNN
-F 2 "IWconnectors:PIN_ARRAY_14x2" H 18900 4850 50  0001 C CNN
-F 3 "" H 18550 4700 60  0000 C CNN
-	1    18550 4700
+P 20000 1100
+F 0 "XS10" H 20250 1450 71  0000 L CNN
+F 1 "PBD-28" H 20150 1350 71  0000 L CNN
+F 2 "IWconnectors:PIN_ARRAY_14x2" H 20350 1250 50  0001 C CNN
+F 3 "" H 20000 1100 60  0000 C CNN
+	1    20000 1100
 	1    0    0    -1
 $EndComp

Commit message: Добавил в схему различные варианты подключения резистора регулировки контрастности для графического дисплея.
Parts:
- added R10, R13, R16, R7: 0, IWsmd_case:SMD0603, symbol LFresistor:RESISTOR
Connections:
- wire segments 488 -> 499
Other:
- note added: "10 кОм"
- note added: "100 кОм"
- note added: "20 кОм"
- note added: "D/I"
- note added: "MT-12864A"
- note added: "MT-12864A-...-T"
- note added: "R10"
- note added: "R13"
- note added: "R15"
- note added: "R7"
- note added: "Vdd"
- note added: "Vo"
- note added: "WG12864A"
- note added: "Установка резисторов для регулировки контрастности \n у различных моделей графических дисплеев\n подключаемых к разъёму XP6"
- note added: "есть"
- note added: "нет"
- moved on the sheet: R15
Changed lines of the file:
@@
 	21000 12600 21450 12600
 Wire Wire Line
-	20550 12200 21450 12200
-Wire Wire Line
-	19800 12300 20300 12300
-Wire Wire Line
 	21000 12100 21450 12100
 Wire Wire Line
 	21000 12000 21450 12000
-Wire Wire Line
-	20550 12300 20850 12300
 Wire Wire Line
 	21000 13800 21450 13800
@@
 	21000 9750 21450 9750
 Wire Wire Line
-	19750 9950 20200 9950
+	19300 9950 19750 9950
 Wire Wire Line
 	20450 9850 21450 9850
@@
 Text Label 21000 10650 0    60   ~ 0
 PJ2
-Text Label 19800 12300 0    60   ~ 0
+Text Label 18750 12650 0    60   ~ 0
 MPU_VCC
 Text Label 21000 13700 0    60   ~ 0
 V_OUT
-Text Label 20850 12300 2    60   ~ 0
+Text Label 20650 12650 2    60   ~ 0
 V_OUT
 Text Label 21400 14300 2    60   ~ 0
@@
 GND
 Text Notes 21900 12150 0    60   ~ 0
-VCC
+Vdd
 Text Notes 21900 12250 0    60   ~ 0
-VEE
+Vo
 Text Notes 21900 12350 0    60   ~ 0
-RS
+D/I
 Text Notes 21900 12450 0    60   ~ 0
 R/W
@@
 L LFresistor:RESISTOR_TRIMMING R15
 U 1 1 525BB8BD
-P 20300 12300
-F 0 "R15" H 20450 12600 71  0000 C CNN
-F 1 "20к" H 20450 12500 71  0000 C CNN
-F 2 "IWcomponents:Electron_3296W" H 20300 12300 60  0001 C CNN
-F 3 "" H 20300 12300 60  0001 C CNN
-	1    20300 12300
+P 19750 12650
+F 0 "R15" H 19900 12950 71  0000 C CNN
+F 1 "20к" H 19900 12850 71  0000 C CNN
+F 2 "IWcomponents:Electron_3296W" H 19750 12650 60  0001 C CNN
+F 3 "" H 19750 12650 60  0001 C CNN
+	1    19750 12650
 	1    0    0    -1
 $EndComp
@@
 Text Label 20700 9950 2    60   ~ 0
 GND
-Text Label 19750 9950 0    60   ~ 0
+Text Label 19300 9950 0    60   ~ 0
 MPU_VCC
 $Comp
@@
 Wire Wire Line
 	9200 10150 10550 10150
+$Comp
+L LFresistor:RESISTOR R7
+U 1 1 63B31167
+P 19300 12650
+F 0 "R7" H 19300 12750 71  0000 C CNN
+F 1 "0" H 19550 12750 71  0000 C CNN
+F 2 "IWsmd_case:SMD0603" H 19300 12650 60  0001 C CNN
+F 3 "" H 19300 12650 60  0001 C CNN
+	1    19300 12650
+	1    0    0    -1
+$EndComp
+Wire Wire Line
+	18750 12650 19300 12650
+Wire Wire Line
+	19550 12650 19650 12650
+$Comp
+L LFresistor:RESISTOR R13
+U 1 1 63E41378
+P 19750 12200
+F 0 "R13" H 19750 12350 71  0000 C CNN
+F 1 "0" H 20000 12350 71  0000 C CNN
+F 2 "IWsmd_case:SMD0603" H 19750 12200 60  0001 C CNN
+F 3 "" H 19750 12200 60  0001 C CNN
+	1    19750 12200
+	1    0    0    -1
+$EndComp
+Wire Wire Line
+	20000 12550 20100 12550
+Wire Wire Line
+	20100 12550 20100 12200
+$Comp
+L LFresistor:RESISTOR R10
+U 1 1 6428DAB0
+P 19300 13000
+F 0 "R10" H 19300 13100 71  0000 C CNN
+F 1 "0" H 19550 13100 71  0000 C CNN
+F 2 "IWsmd_case:SMD0603" H 19300 13000 60  0001 C CNN
+F 3 "" H 19300 13000 60  0001 C CNN
+	1    19300 13000
+	1    0    0    -1
+$EndComp
+Wire Wire Line
+	19650 12650 19650 13000
+Wire Wire Line
+	19650 13000 19550 13000
+Connection ~ 19650 12650
+Wire Wire Line
+	19650 12650 19750 12650
+Wire Wire Line
+	18750 13000 19300 13000
+Text Label 18750 13000 0    60   ~ 0
+GND
+Wire Wire Line
+	20000 12200 20100 12200
+Connection ~ 20100 12200
+Wire Wire Line
+	19750 12200 19650 12200
+Wire Wire Line
+	19650 12200 19650 12650
+Wire Wire Line
+	20100 12200 21450 12200
+Wire Wire Line
+	20000 12650 20650 12650
+Text Notes 16350 12400 0    50   ~ 0
+Установка резисторов для  регулировки контрастности \n     у различных моделей графических дисплеев\n          подключаемых к разъёму XP6
+Text Notes 16350 12700 0    50   ~ 0
+WG12864A
+Text Notes 16350 12850 0    50   ~ 0
+MT-12864A
+Text Notes 16200 13000 0    50   ~ 0
+MT-12864A-...-T
+Wire Notes Line
+	16150 12750 18400 12750
+Wire Notes Line
+	16150 12900 18400 12900
+Wire Notes Line
+	17300 12450 17300 13050
+Wire Notes Line
+	17650 12450 17650 13050
+Wire Notes Line
+	18000 12450 18000 13050
+Wire Notes Line
+	16150 12600 18400 12600
+Text Notes 17050 12550 0    50   ~ 0
+R7
+Text Notes 17400 12550 0    50   ~ 0
+R10
+Text Notes 17750 12550 0    50   ~ 0
+R13
+Text Notes 17050 12700 0    50   ~ 0
+есть
+Text Notes 17400 12700 0    50   ~ 0
+нет
+Text Notes 17750 12700 0    50   ~ 0
+нет
+Text Notes 17750 12850 0    50   ~ 0
+есть
+Text Notes 17400 12850 0    50   ~ 0
+нет
+Text Notes 17050 12850 0    50   ~ 0
+нет
+Text Notes 17050 13000 0    50   ~ 0
+нет
+Text Notes 17750 13000 0    50   ~ 0
+нет
+Text Notes 17400 13000 0    50   ~ 0
+есть
+Wire Notes Line
+	16150 12600 16150 13050
+Wire Notes Line
+	16150 13050 18400 13050
+Wire Notes Line
+	16950 12450 18400 12450
+Wire Notes Line
+	16950 12450 16950 13050
+Text Notes 18100 12550 0    50   ~ 0
+R15
+Text Notes 18050 12700 0    50   ~ 0
+20 кОм
+Text Notes 18050 12850 0    50   ~ 0
+10 кОм
+Text Notes 18050 13000 0    50   ~ 0
+100 кОм
+Wire Notes Line
+	18400 12450 18400 13050
+$Comp
+L LFresistor:RESISTOR R16
+U 1 1 65C8A68B
+P 19750 9950
+F 0 "R16" H 19750 10100 71  0000 C CNN
+F 1 "0" H 20000 10100 71  0000 C CNN
+F 2 "IWsmd_case:SMD0603" H 19750 9950 60  0001 C CNN
+F 3 "" H 19750 9950 60  0001 C CNN
+	1    19750 9950
+	1    0    0    -1
+$EndComp
+Wire Wire Line
+	20200 9950 20000 9950
 $EndSCHEMATC
